File: Part 3 - Improving clock options/Clock.kicad_sch (KiCad schematic)
At the start: 19 parts, among them SW4 STEP, U3 LMC555, U4 74HC14, U5 74HC74

Commit message: Worked on Part 3's clock
Parts:
- removed C2, C3, C4, C5, C6: 0.1µF, Capacitor_THT:C_Disc_D3.0mm_W1.6mm_P2.50mm, symbol Device:C
- added C? (x7): 0.1µF, Capacitor_THT:C_Disc_D3.0mm_W1.6mm_P2.50mm, symbol Device:C
- added C? (x2): 1µF, Capacitor_THT:C_Disc_D3.0mm_W1.6mm_P2.50mm, symbol Device:C
- added D?: CLOCK, LED_THT:LED_D3.0mm, symbol Device:LED
- added D?: SLOW, LED_THT:LED_D3.0mm, symbol Device:LED
- added D?: FAST, LED_THT:LED_D3.0mm, symbol Device:LED
- added D?: RUN, LED_THT:LED_D3.0mm, symbol Device:LED
- added R? (x2): 22KΩ, Resistor_THT:R_Axial_DIN0207_L6.3mm_D2.5mm_P7.62mm_Horizontal, symbol Device:R_US
- added R? (x4): 330Ω, Resistor_THT:R_Axial_DIN0207_L6.3mm_D2.5mm_P10.16mm_Horizontal, symbol Device:R_US
- added R? (x2): 1KΩ, Resistor_THT:R_Axial_DIN0207_L6.3mm_D2.5mm_P7.62mm_Horizontal, symbol Device:R_US
- added R? (x4): 3K3Ω, Resistor_THT:R_Axial_DIN0207_L6.3mm_D2.5mm_P7.62mm_Horizontal, symbol Device:R_US
- added R?: 3K3Ω, Resistor_THT:R_Axial_DIN0207_L6.3mm_D2.5mm_P10.16mm_Horizontal, symbol Device:R_US
- added RN?: 3K3Ω, Resistor_THT:R_Array_SIP5, symbol Device:R_Network04_US
- added SW?: BOOT SPEED, symbol Switch:SW_SPDT
- added SW?: MODE, Button_Switch_THT:SW_PUSH_6mm, symbol Switch:SW_Push
- added SW?: SPEED, Button_Switch_THT:SW_PUSH_6mm, symbol Switch:SW_Push
- added SW?: SW_DIP_x04, symbol Switch:SW_DIP_x04
- added SW?: BOOT MODE, symbol Switch:SW_SPDT
- added U?: 74HC193, symbol 74xx:74LS193
- added U?: 74HC151, symbol 74xx:74LS151
- added U? (x3): 74HC74, Package_DIP:DIP-14_W7.62mm_Socket, symbol 74xx:74HC74
- added U? (x3): 74HC14, Package_DIP:DIP-14_W7.62mm_Socket, symbol 74xx:74HC14
- added X?: CXO_DIP8, Oscillator:Oscillator_DIP-8, symbol Oscillator:CXO_DIP8
- D?: renamed from D3; value CLK -> STEP
- R?: renamed from R11; value 10KΩ -> 330Ω
- renumbered C8 to C?, C7 to C?, C9 to C?, R9 to R?, R10 to R?, R13 to R?, R12 to R?, RV1 to RV?, SW4 to SW?, U5 to U?, U3 to U?, U4 to U?
Connections:
- net +5V: now also C?.1, C?.1, C?.1, C?.1, C?.1, C?.1, C?.1, R?.1, R?.1, R?.2, R?.2, R?.2, R?.2, SW?.1, SW?.2, SW?.3, SW?.4, U?.10 (~{S}), U?.11 (S0), U?.13 (~{R}), U?.14 (VCC), U?.16 (VCC), U?.16 (VCC), U?.5 (UP), X?.1 (EN), X?.8 (Vcc); no longer U?.10 (~{S}), U?.11 (C), U?.12 (D), U?.13 (~{R})
- net GND: now also C?.2, C?.2, C?.2, C?.2, C?.2, C?.2, C?.2, C?.2, C?.2, D?.1 (K), D?.1 (K), D?.1 (K), D?.1 (K), R?.2, RN?.1 (common), SW?.2, SW?.2, U?.14 (CLR), U?.7 (GND), U?.8 (GND), U?.8 (GND), X?.4 (GND)
- net SLOW: now also U?.3 (I1), U?.4 (I0)
- net STEP: now also U?.12 (I7), U?.13 (I6), U?.14 (I5), U?.15 (I4)
- net MODE: now reaches R?.1
- net MODE: now also U?.5 (Q), U?.9 (S2)
- net at R?.2, SW?.1: now also R?.2; no longer R?.1
- net at C?.1, U?.1: now also R?.1; no longer R?.2
- new net: C?.1, R?.1, U?.5
- new net: R?.2, R?.2, SW?.1 (x2)
- new net: R?.1, U?.2 (D), U?.6 (~{Q})
- new net: D?.2 (A), R?.2 (x4)
- new net: RN?.3 (R2), SW?.7, U?.1 (B)
- new net: RN?.4 (R3), SW?.6, U?.10 (C)
- new net: U?.11 (C), U?.11 (~{LOAD}), U?.13 (~{BO})
- new net: RN?.2 (R1), SW?.8, U?.15 (A)
- new net: U?.4 (DOWN), X?.5 (OUT)
- new net: RN?.5 (R4), SW?.5, U?.9 (D)
- new net: R?.1, SW?.1 (A), U?.13 (~{R})
- new net: R?.1, SW?.3 (C), U?.10 (~{S})
- new net: C?.1, R?.1, U?.3
- new net: R?.1, U?.8
- new net: R?.1, SW?.1 (A), U?.1 (~{R})
- new net: R?.1, SW?.3 (C), U?.4 (~{S})
- new net: U?.12 (D), U?.8 (~{Q})
- new net: U?.11 (C), U?.6
- new net: R?.1, U?.12 (D), U?.8 (~{Q})
- new net: U?.3 (C), U?.4
- new net CLK: U?.5 (Z)
- new net FAST: U?.1 (I3), U?.2 (I2), U?.9 (Q)
- new net PWR_UP: SW?.2 (B), SW?.2 (B)
- new net SPEED: R?.1, U?.10 (S1), U?.9 (Q)
- new net ~{CLK_EN}: R?.1, U?.7 (~{E})
- new net ~{CLK}: U?.6 (~{Z}), U?.9
- no-connect marks 3 -> 6
Other:
- note added: "CLOCK OUTPUT"
- note added: "FAST CLOCK"
- note added: "MODE: STEP/RUN"
- note added: "SINGLE STEP"
- note added: "SLOW CLOCK"
- note added: "SPEED: SLOW/FAST"
- note removed: "Blue"
- moved on the sheet: C?, D?, R?, RV?, SW?, U?, U?A, U?C, U?G
