File: Part 3 - Improving clock options/Part 3 - Improving clock options.kicad_sch (KiCad schematic)
At the start: 0 parts

Commit message: Worked on Part 3's clock
Other:
- sheet Clock ports: added CLK, ~{CLK_EN}; removed none
- sheet Reset ports: added CLK, PWR_UP, ~{M_RST}, ~{PWR_UP}, ~{RESET}; removed none
