File: Part 3 - Improving clock options/Power.kicad_sch (KiCad schematic)
At the start: 11 parts, among them J1 +5V DC CP, Q1 IPP80P03P4L, Q2 PN2222A, SW1 POWER

Commit message: Worked on Part 3's clock
Parts:
- renumbered C1 to C?, D1 to D?, J1 to J?, Q2 to Q?, Q1 to Q?, R2 to R?, R1 to R?, R4 to R?, R3 to R?, R5 to R?, SW1 to SW?
Changed lines of the file:
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@@
   (symbol (lib_id "Transistor_BJT:PN2222A") (at 97.79 101.6 0) (mirror y) (unit 1)
     (in_bom yes) (on_board yes)
-    (property "Reference" "Q2" (id 0) (at 92.9386 100.4316 0)
+    (property "Reference" "Q?" (id 0) (at 92.9386 100.4316 0)
       (effects (font (size 1.27 1.27)) (justify left))
     )
@@
   (symbol (lib_id "Connector:Barrel_Jack") (at 39.37 59.69 0) (unit 1)
     (in_bom yes) (on_board yes)
-    (property "Reference" "J1" (id 0) (at 33.02 58.42 0)
+    (property "Reference" "J?" (id 0) (at 33.02 58.42 0)
       (effects (font (size 1.27 1.27)) (justify right))
     )
@@
   (symbol (lib_id "Transistor_FET:IRF4905") (at 116.84 64.77 0) (mirror x) (unit 1)
     (in_bom yes) (on_board yes)
-    (property "Reference" "Q1" (id 0) (at 122.047 63.6016 0)
+    (property "Reference" "Q?" (id 0) (at 122.047 63.6016 0)
       (effects (font (size 1.27 1.27)) (justify left))
     )
@@
   (symbol (lib_id "Device:R_US") (at 95.25 73.66 180) (unit 1)
     (in_bom yes) (on_board yes)
-    (property "Reference" "R2" (id 0) (at 92.71 72.39 0)
+    (property "Reference" "R?" (id 0) (at 92.71 72.39 0)
       (effects (font (size 1.27 1.27)) (justify left))
     )
@@
   (symbol (lib_id "Device:R_US") (at 85.09 71.12 180) (unit 1)
     (in_bom yes) (on_board yes)
-    (property "Reference" "R1" (id 0) (at 82.55 69.85 0)
+    (property "Reference" "R?" (id 0) (at 82.55 69.85 0)
       (effects (font (size 1.27 1.27)) (justify left))
     )
@@
   (symbol (lib_id "Switch:SW_Push") (at 64.77 77.47 90) (mirror x) (unit 1)
     (in_bom yes) (on_board yes)
-    (property "Reference" "SW1" (id 0) (at 60.96 76.2 90)
+    (property "Reference" "SW?" (id 0) (at 60.96 76.2 90)
       (effects (font (size 1.27 1.27)) (justify left))
     )
@@
   (symbol (lib_id "Device:R_US") (at 105.41 93.98 180) (unit 1)
     (in_bom yes) (on_board yes)
-    (property "Reference" "R4" (id 0) (at 102.87 92.71 0)
+    (property "Reference" "R?" (id 0) (at 102.87 92.71 0)
       (effects (font (size 1.27 1.27)) (justify left))
     )
@@
   (symbol (lib_id "Device:R_US") (at 80.01 87.63 90) (unit 1)
     (in_bom yes) (on_board yes)
-    (property "Reference" "R3" (id 0) (at 80.01 82.55 90))
+    (property "Reference" "R?" (id 0) (at 80.01 82.55 90))
     (property "Value" "1MΩ" (id 1) (at 80.01 85.09 90))
     (property "Footprint" "Resistor_THT:R_Axial_DIN0207_L6.3mm_D2.5mm_P10.16mm_Horizontal" (id 2) (at 80.264 86.614 90)
@@
   (symbol (lib_id "Device:C") (at 64.77 96.52 0) (mirror y) (unit 1)
     (in_bom yes) (on_board yes)
-    (property "Reference" "C1" (id 0) (at 61.849 95.3516 0)
+    (property "Reference" "C?" (id 0) (at 61.849 95.3516 0)
       (effects (font (size 1.27 1.27)) (justify left))
     )
@@
   (symbol (lib_id "Device:R_US") (at 119.38 99.06 180) (unit 1)
     (in_bom yes) (on_board yes)
-    (property "Reference" "R5" (id 0) (at 116.84 97.79 0)
+    (property "Reference" "R?" (id 0) (at 116.84 97.79 0)
       (effects (font (size 1.27 1.27)) (justify left))
     )
@@
   (symbol (lib_id "power:+5V") (at 138.43 68.58 0) (unit 1)
     (in_bom yes) (on_board yes)
-    (property "Reference" "#PWR01" (id 0) (at 138.43 72.39 0)
+    (property "Reference" "#PWR?" (id 0) (at 138.43 72.39 0)
       (effects (font (size 1.27 1.27)) hide)
     )
@@
   (symbol (lib_id "power:PWR_FLAG") (at 139.7 74.93 270) (unit 1)
     (in_bom yes) (on_board yes)
-    (property "Reference" "#FLG01" (id 0) (at 141.605 74.93 0)
+    (property "Reference" "#FLG?" (id 0) (at 141.605 74.93 0)
       (effects (font (size 1.27 1.27)) hide)
     )
@@
   (symbol (lib_id "power:PWR_FLAG") (at 139.7 109.22 270) (unit 1)
     (in_bom yes) (on_board yes)
-    (property "Reference" "#FLG02" (id 0) (at 141.605 109.22 0)
+    (property "Reference" "#FLG?" (id 0) (at 141.605 109.22 0)
       (effects (font (size 1.27 1.27)) hide)
     )
@@
   (symbol (lib_id "power:GND") (at 138.43 114.3 0) (unit 1)
     (in_bom yes) (on_board yes)
-    (property "Reference" "#PWR02" (id 0) (at 138.43 120.65 0)
+    (property "Reference" "#PWR?" (id 0) (at 138.43 120.65 0)
       (effects (font (size 1.27 1.27)) hide)
     )
@@
   (symbol (lib_id "Device:LED") (at 119.38 83.82 90) (unit 1)
     (in_bom yes) (on_board yes)
-    (property "Reference" "D1" (id 0) (at 122.3772 82.8294 90)
+    (property "Reference" "D?" (id 0) (at 122.3772 82.8294 90)
       (effects (font (size 1.27 1.27)) (justify right))
     )
