File: Part 3 - Improving clock options/Reset.kicad_sch (KiCad schematic)
At the start: 7 parts, among them SW2 RESET, U2 74LS175

Commit message: Worked on Part 3's clock
Parts:
- added C? (x2): 0.1µF, Capacitor_THT:C_Disc_D3.0mm_W1.6mm_P2.50mm, symbol Device:C
- added U? (x2): 74HC14, Package_DIP:DIP-14_W7.62mm_Socket, symbol 74xx:74HC14
- renumbered C1 to C?, D2 to D?, R2 to R?, R8 to R?, RS1 to RS?, SW2 to SW?, U2 to U?
Connections:
- net +5V: now also C?.1, C?.1
- net GND: now also C?.2, C?.2
- net at C?.1, R?.1, RS?.2 (VCC): now also U?.13
- net ~{M_RST}: now reaches RS?.1 (~{RESET}), SW?.1, U?.1 (~{Mr}), U?.4 (D0)
- new net PWR_UP: U?.10
- new net ~{PWR_UP}: U?.11, U?.12
Other:
- note added: "Bypass capacitors"
