File: Part 2 - Improving clock options/Clock.kicad_sch (KiCad schematic)
At the start: 58 parts

Commit message: Finished clock in part 2, added part 3
Parts:
- removed RN?: 3K3Ω, Resistor_THT:R_Array_SIP5, symbol Device:R_Network04_US
- removed SW?: SW_DIP_x04, symbol Switch:SW_DIP_x04
- removed U?: 74HC193, symbol 74xx:74LS193
- R5, R7, R9: renamed from R?; value 22KΩ -> 20KΩ
- RV1: renamed from RV?; footprint Potentiometer_THT:Potentiometer_Bourns_3296W_Vertical -> Potentiometer_THT:Potentiometer_Bourns_3386P_Vertical; symbol Part-1---Testing-the-Z80-rescue:R_POT_US-Device -> Device:R_Potentiometer_US
- U4: renamed from U?; symbol 0_Fred's_Local_Library:LMC555 -> 0_Z80_Library:LMC555
- X1: renamed from X?; value CXO_DIP8 -> 14.7456MHz
- gave numbers to parts that had none: 41
Connections:
- net at U5.11 (C): now also X1.5 (OUT)
- net at R14.1, U3.1 (~{R}): now also SW6.3 (C); no longer SW6.1 (A)
- net at R10.1, U3.4 (~{S}): now also SW6.1 (A); no longer SW6.3 (C)
- net ~{CLK_EN}: no longer names the net of R20.1, U7.7 (~{E})
- net ~{CLK}: no longer names the net of U1.9, U7.6 (~{Z})
- no-connect marks 6 -> 1
Other:
- note added: "MODE: STEP/FREERUN"
- note removed: "MODE: STEP/RUN"
- moved on the sheet: D7, R21, U1G, U3C, U5B, U5C, X1
