File: Part 7 - Keyboard/Part 7 - Keyboard.kicad_pcb (KiCad board)
At the start: 2 copper layers, 333.4 x 124.5 mm, 98 parts, among them J1 KEYBOARD, SW1 0, SW10 9, SW11 MINUS, SW12 EQUALS, SW13 BACK_SLASH, SW14 LEFT_BRACKET, SW15 RIGHT_BRACKET, SW16 SEMICOLON, SW17 QUOTE, SW18 TILDE, SW19 COMMA, SW2 1, SW20 PERIOD, SW21 SLASH, SW22 DEAD, SW23 A, SW24 B, SW25 C, SW26 D, SW27 E, SW28 F, SW29 G, SW3 2, SW30 H, SW31 I, SW32 J, SW33 K, SW34 L, SW35 M, SW36 N, SW37 O, SW38 P, SW39 Q, SW4 3, SW40 R, SW41 S, SW42 T, SW43 U, SW44 V, SW45 W, SW46 X, SW47 Y, SW48 Z, SW49 SHIFT, SW5 4, SW50 CTRL, SW51 GRAPH, SW52 CAPS_LOCK, SW53 CODE/KANA, SW54 F1/F6, SW55 F2/F7, SW56 F3/F8, SW57 F4/F9, SW58 F5/F10, SW59 ESC, SW6 5, SW60 TAB, SW61 STOP, SW62 BACK_SPACE, SW63 SELECT, SW64 RETURN, SW65 SPACE, SW66 HOME/CLS, SW67 INSERT, SW68 DELETE, SW69 LEFT, SW7 6, SW70 UP, SW71 DOWN, SW72 RIGHT, SW73 SHIFT, SW8 7, SW9 8, U1 74LS145, U2 74LS07

Commit message: Added Keyboard, and minor fixes
Parts:
- removed HOLE1, HOLE2, HOLE3, HOLE4, HOLE5, HOLE6, HOLE7: HOLE, My_Components:Hole_3mm
- removed REF**: OSHW-Logo_7.5x8mm_SilkScreen, Symbol:OSHW-Logo_7.5x8mm_SilkScreen
- removed REF**: Symbol_GNU-Logo_SilkscreenTop, Symbol:Symbol_GNU-Logo_SilkscreenTop
- added H1: MH, MountingHole:MountingHole_3.2mm_M3_Pad_Via, F.Cu at (41.8, 41.5)
- added H2: MountingHole_Pad, MountingHole:MountingHole_3.2mm_M3_Pad_Via, F.Cu at (41.8, 153.3)
- added H3: MountingHole_Pad, MountingHole:MountingHole_3.2mm_M3_Pad_Via, F.Cu at (176.4, 41.5)
- added H4: MountingHole_Pad, MountingHole:MountingHole_3.2mm_M3_Pad_Via, F.Cu at (176.4, 153.3)
- added H5: MountingHole_Pad, MountingHole:MountingHole_3.2mm_M3_Pad_Via, F.Cu at (280.5, 153.3)
- added H6: MountingHole_Pad, MountingHole:MountingHole_3.2mm_M3_Pad_Via, F.Cu at (302.1, 72.0)
- added H7: MountingHole_Pad, MountingHole:MountingHole_3.2mm_M3_Pad_Via, F.Cu at (331.3, 110.1)
- added REF3: OSHW-Symbol_8.9x8mm_SilkScreen, Symbol:OSHW-Symbol_8.9x8mm_SilkScreen, B.Cu at (335.1, 130.4)
- added REF4: OSHW-Symbol_8.9x8mm_SilkScreen, Symbol:OSHW-Symbol_8.9x8mm_SilkScreen, F.Cu at (335.1, 130.5)
- C1: renamed from C3; footprint My_Components:Cap_Tant_508 -> Capacitor_THT:CP_Radial_D5.0mm_P2.50mm
- C2: footprint My_Components:Cap_Cer_508 -> Capacitor_THT:C_Disc_D3.0mm_W2.0mm_P2.50mm
- C3: renamed from C1; footprint My_Components:Cap_Cer_508 -> Capacitor_THT:C_Disc_D3.0mm_W2.0mm_P2.50mm
- D1: footprint My_Components:LED_3mm -> LED_THT:LED_D3.0mm
- D2: value CAPS -> KANA; footprint Cherry_MX:CHERRY_MX_LED -> LED_THT:LED_D3.0mm
- D3: value KANA -> CAPS; footprint Cherry_MX:CHERRY_MX_LED -> LED_THT:LED_D3.0mm
- D4, D5, D6: footprint My_Components:Diode_762 -> Diode_THT:D_DO-35_SOD27_P7.62mm_Horizontal
- J1: footprint My_Components:Conn_Pin_Header_8x2_2.54mm -> Connector_PinSocket_2.54mm:PinSocket_2x08_P2.54mm_Vertical
- R1, R2, R3: value 470 -> 330; footprint My_Components:Res_762 -> Resistor_THT:R_Axial_DIN0204_L3.6mm_D1.6mm_P7.62mm_Horizontal
- RN1: value 4.7k -> 3K3; footprint My_Components:Conn_SIL6 -> Resistor_THT:R_Array_SIP5
- SW1: renamed from SW73; footprint Cherry_MX:CHERRY_PCB_275H -> 0_Z80_Library:SW_Cherry_MX_2.75u_PCB
- SW10: renamed from SW65; footprint Cherry_MX:CHERRY_PCB_625H -> 0_Z80_Library:SW_Cherry_MX_6.25u_PCB
- SW11: renamed from SW2; footprint Cherry_MX:CHERRY_PCB_100H -> 0_Z80_Library:SW_Cherry_MX_1.00u_PCB
- SW12: renamed from SW10; footprint Cherry_MX:CHERRY_PCB_100H -> 0_Z80_Library:SW_Cherry_MX_1.00u_PCB
- SW13: renamed from SW18; footprint Cherry_MX:CHERRY_PCB_100H -> 0_Z80_Library:SW_Cherry_MX_1.00u_PCB
- SW14: renamed from SW26; footprint Cherry_MX:CHERRY_PCB_100H -> 0_Z80_Library:SW_Cherry_MX_1.00u_PCB
- SW15: renamed from SW34; footprint Cherry_MX:CHERRY_PCB_100H -> 0_Z80_Library:SW_Cherry_MX_1.00u_PCB
- SW16: renamed from SW42; footprint Cherry_MX:CHERRY_PCB_100H -> 0_Z80_Library:SW_Cherry_MX_1.00u_PCB
- SW17: renamed from SW50; footprint Cherry_MX:CHERRY_PCB_125H -> 0_Z80_Library:SW_Cherry_MX_1.25u_PCB
- SW18: renamed from SW58; footprint Cherry_MX:CHERRY_PCB_100H -> 0_Z80_Library:SW_Cherry_MX_1.00u_PCB
- SW19: renamed from SW66; footprint Cherry_MX:CHERRY_PCB_100H -> 0_Z80_Library:SW_Cherry_MX_1.00u_PCB
- SW2: renamed from SW1; footprint Cherry_MX:CHERRY_PCB_100H -> 0_Z80_Library:SW_Cherry_MX_1.00u_PCB
- SW20: renamed from SW3; footprint Cherry_MX:CHERRY_PCB_100H -> 0_Z80_Library:SW_Cherry_MX_1.00u_PCB
- SW21: renamed from SW11; footprint Cherry_MX:CHERRY_PCB_100H -> 0_Z80_Library:SW_Cherry_MX_1.00u_PCB
- SW22: renamed from SW19; footprint Cherry_MX:CHERRY_PCB_100H -> 0_Z80_Library:SW_Cherry_MX_1.00u_PCB
- SW23: renamed from SW27; footprint Cherry_MX:CHERRY_PCB_100H -> 0_Z80_Library:SW_Cherry_MX_1.00u_PCB
- SW24: renamed from SW35; footprint Cherry_MX:CHERRY_PCB_100H -> 0_Z80_Library:SW_Cherry_MX_1.00u_PCB
- SW25: renamed from SW43; footprint Cherry_MX:CHERRY_PCB_100H -> 0_Z80_Library:SW_Cherry_MX_1.00u_PCB
- SW26: renamed from SW51; footprint Cherry_MX:CHERRY_PCB_125H -> 0_Z80_Library:SW_Cherry_MX_1.25u_PCB
- SW27: renamed from SW59; footprint Cherry_MX:CHERRY_PCB_100H -> 0_Z80_Library:SW_Cherry_MX_1.00u_PCB
- SW28: renamed from SW67; footprint Cherry_MX:CHERRY_PCB_100H -> 0_Z80_Library:SW_Cherry_MX_1.00u_PCB
- SW29: renamed from SW4; footprint Cherry_MX:CHERRY_PCB_100H -> 0_Z80_Library:SW_Cherry_MX_1.00u_PCB
- SW3: renamed from SW9; footprint Cherry_MX:CHERRY_PCB_100H -> 0_Z80_Library:SW_Cherry_MX_1.00u_PCB
- SW30: renamed from SW12; value EQUALS -> EQUAL; footprint Cherry_MX:CHERRY_PCB_100H -> 0_Z80_Library:SW_Cherry_MX_1.00u_PCB
- SW31: renamed from SW20; footprint Cherry_MX:CHERRY_PCB_100H -> 0_Z80_Library:SW_Cherry_MX_1.00u_PCB
- SW32: renamed from SW28; footprint Cherry_MX:CHERRY_PCB_100H -> 0_Z80_Library:SW_Cherry_MX_1.00u_PCB
- SW33: renamed from SW36; footprint Cherry_MX:CHERRY_PCB_100H -> 0_Z80_Library:SW_Cherry_MX_1.00u_PCB
- SW34: renamed from SW44; footprint Cherry_MX:CHERRY_PCB_100H -> 0_Z80_Library:SW_Cherry_MX_1.00u_PCB
- SW35: renamed from SW52; value CAPS_LOCK -> CAPS LOCK; footprint Cherry_MX:CHERRY_PCB_175H -> 0_Z80_Library:SW_Cherry_MX_1.75u_PCB
- SW36: renamed from SW60; footprint Cherry_MX:CHERRY_PCB_150H -> 0_Z80_Library:SW_Cherry_MX_1.50u_PCB
- SW37: renamed from SW68; footprint Cherry_MX:CHERRY_PCB_100H -> 0_Z80_Library:SW_Cherry_MX_1.00u_PCB
- SW38: renamed from SW5; footprint Cherry_MX:CHERRY_PCB_100H -> 0_Z80_Library:SW_Cherry_MX_1.00u_PCB
- SW39: renamed from SW13; value BACK_SLASH -> BACKSLASH; footprint Cherry_MX:CHERRY_PCB_150H -> 0_Z80_Library:SW_Cherry_MX_1.50u_PCB
- SW4: renamed from SW17; footprint Cherry_MX:CHERRY_PCB_100H -> 0_Z80_Library:SW_Cherry_MX_1.00u_PCB
- SW40: renamed from SW21; footprint Cherry_MX:CHERRY_PCB_100H -> 0_Z80_Library:SW_Cherry_MX_1.00u_PCB
- SW41: renamed from SW29; footprint Cherry_MX:CHERRY_PCB_100H -> 0_Z80_Library:SW_Cherry_MX_1.00u_PCB
- SW42: renamed from SW37; footprint Cherry_MX:CHERRY_PCB_100H -> 0_Z80_Library:SW_Cherry_MX_1.00u_PCB
- SW43: renamed from SW45; footprint Cherry_MX:CHERRY_PCB_100H -> 0_Z80_Library:SW_Cherry_MX_1.00u_PCB
- SW44: renamed from SW53; footprint Cherry_MX:CHERRY_PCB_125H -> 0_Z80_Library:SW_Cherry_MX_1.25u_PCB
- SW45: renamed from SW61; footprint Cherry_MX:CHERRY_PCB_100H -> 0_Z80_Library:SW_Cherry_MX_1.00u_PCB
- SW46: renamed from SW69; footprint Cherry_MX:CHERRY_PCB_100H -> 0_Z80_Library:SW_Cherry_MX_1.00u_PCB
- SW47: renamed from SW6; footprint Cherry_MX:CHERRY_PCB_100H -> 0_Z80_Library:SW_Cherry_MX_1.00u_PCB
- SW48: renamed from SW14; value LEFT_BRACKET -> LEFT BRACKET; footprint Cherry_MX:CHERRY_PCB_100H -> 0_Z80_Library:SW_Cherry_MX_1.00u_PCB
- SW49: renamed from SW22; footprint Cherry_MX:CHERRY_PCB_125H -> 0_Z80_Library:SW_Cherry_MX_1.25u_PCB
- SW5: renamed from SW25; footprint Cherry_MX:CHERRY_PCB_100H -> 0_Z80_Library:SW_Cherry_MX_1.00u_PCB
- SW50: renamed from SW30; footprint Cherry_MX:CHERRY_PCB_100H -> 0_Z80_Library:SW_Cherry_MX_1.00u_PCB
- SW51: renamed from SW38; footprint Cherry_MX:CHERRY_PCB_100H -> 0_Z80_Library:SW_Cherry_MX_1.00u_PCB
- SW52: renamed from SW46; footprint Cherry_MX:CHERRY_PCB_100H -> 0_Z80_Library:SW_Cherry_MX_1.00u_PCB
- SW53: renamed from SW54; footprint Cherry_MX:CHERRY_PCB_100H -> 0_Z80_Library:SW_Cherry_MX_1.00u_PCB
- SW54: renamed from SW62; value BACK_SPACE -> BACKSPACE; footprint Cherry_MX:CHERRY_PCB_200H -> 0_Z80_Library:SW_Cherry_MX_2.00u_PCB
- SW55: renamed from SW70; footprint Cherry_MX:CHERRY_PCB_100H -> 0_Z80_Library:SW_Cherry_MX_1.00u_PCB
- SW56: renamed from SW7; footprint Cherry_MX:CHERRY_PCB_100H -> 0_Z80_Library:SW_Cherry_MX_1.00u_PCB
- SW57: renamed from SW15; value RIGHT_BRACKET -> RIGHT BRACKET; footprint Cherry_MX:CHERRY_PCB_100H -> 0_Z80_Library:SW_Cherry_MX_1.00u_PCB
- SW58: renamed from SW23; footprint Cherry_MX:CHERRY_PCB_100H -> 0_Z80_Library:SW_Cherry_MX_1.00u_PCB
- SW59: renamed from SW31; footprint Cherry_MX:CHERRY_PCB_100H -> 0_Z80_Library:SW_Cherry_MX_1.00u_PCB
- SW6: renamed from SW33; footprint Cherry_MX:CHERRY_PCB_100H -> 0_Z80_Library:SW_Cherry_MX_1.00u_PCB
- SW60: renamed from SW39; footprint Cherry_MX:CHERRY_PCB_100H -> 0_Z80_Library:SW_Cherry_MX_1.00u_PCB
- SW61: renamed from SW47; footprint Cherry_MX:CHERRY_PCB_100H -> 0_Z80_Library:SW_Cherry_MX_1.00u_PCB
- SW62: renamed from SW55; footprint Cherry_MX:CHERRY_PCB_100H -> 0_Z80_Library:SW_Cherry_MX_1.00u_PCB
- SW63: footprint Cherry_MX:CHERRY_PCB_125H -> 0_Z80_Library:SW_Cherry_MX_1.25u_PCB
- SW64: renamed from SW71; footprint Cherry_MX:CHERRY_PCB_100H -> 0_Z80_Library:SW_Cherry_MX_1.00u_PCB
- SW65: renamed from SW8; footprint Cherry_MX:CHERRY_PCB_100H -> 0_Z80_Library:SW_Cherry_MX_1.00u_PCB
- SW66: renamed from SW16; footprint Cherry_MX:CHERRY_PCB_100H -> 0_Z80_Library:SW_Cherry_MX_1.00u_PCB
- SW67: renamed from SW24; footprint Cherry_MX:CHERRY_PCB_100H -> 0_Z80_Library:SW_Cherry_MX_1.00u_PCB
- SW68: renamed from SW32; footprint Cherry_MX:CHERRY_PCB_100H -> 0_Z80_Library:SW_Cherry_MX_1.00u_PCB
- SW69: renamed from SW40; footprint Cherry_MX:CHERRY_PCB_100H -> 0_Z80_Library:SW_Cherry_MX_1.00u_PCB
- SW7: renamed from SW41; footprint Cherry_MX:CHERRY_PCB_100H -> 0_Z80_Library:SW_Cherry_MX_1.00u_PCB
- SW70: renamed from SW48; footprint Cherry_MX:CHERRY_PCB_100H -> 0_Z80_Library:SW_Cherry_MX_1.00u_PCB
- SW71: renamed from SW56; footprint Cherry_MX:CHERRY_PCB_100H -> 0_Z80_Library:SW_Cherry_MX_1.00u_PCB
- SW72: renamed from SW64; footprint Cherry_MX:CHERRY_PCB_225H -> 0_Z80_Library:SW_Cherry_MX_2.25u_PCB
- SW73: renamed from SW72; footprint Cherry_MX:CHERRY_PCB_100H -> 0_Z80_Library:SW_Cherry_MX_1.00u_PCB
- SW8: renamed from SW49; footprint Cherry_MX:CHERRY_PCB_225H -> 0_Z80_Library:SW_Cherry_MX_2.25u_PCB
- SW9: renamed from SW57; footprint Cherry_MX:CHERRY_PCB_100H -> 0_Z80_Library:SW_Cherry_MX_1.00u_PCB
- U1: value 74LS145 -> 74LS07; footprint My_Components:IC_DIP16_300 -> Package_DIP:DIP-14_W7.62mm_Socket
- U2: value 74LS07 -> 74LS145; footprint My_Components:IC_DIP14_300 -> Package_DIP:DIP-16_W7.62mm_Socket
- moved D2 195.3 mm to (221.7, 57.7)
- moved D3 78.3 mm to (221.7, 48.5)
- moved U2 38.6 mm to (151.1, 59.7), turned to 90 degrees
- moved R3 37.8 mm to (180.5, 59.7)
- moved R1 37.5 mm to (185.3, 59.7)
- moved R2 37.3 mm to (182.9, 59.7)
- moved SW10 28.3 mm to (139.7, 154.6), turned to 180 degrees
- moved D4 28.1 mm to (48.9, 153.0), turned to 90 degrees
- moved D5 28.0 mm to (52.1, 153.0), turned to 90 degrees
- moved D6 27.9 mm to (55.2, 153.0), turned to 90 degrees
- moved J1 23.9 mm to (195.2, 51.7), turned to 90 degrees
- moved RN1 23.4 mm to (199.0, 59.7)
- moved C3 20.9 mm to (147.2, 54.6)
- moved C2 20.9 mm to (147.2, 41.9)
- moved SW61 18.4 mm to (147.2, 87.6)
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Connections:
- net /COLUMN1 renamed /COL1
- net /COLUMN3 renamed /COL3
- net /COLUMN5 renamed /COL5
- net /COLUMN6 renamed /COL6
- net /COLUMN7 renamed /COL7
- D1 pad 1: GND -> Net-(D1-Pad1)
- D1 pad 2: /D1+ -> VCC
- D2 pad 1: /CAPS_LED_BUFFERED -> Net-(D2-Pad1)
- D2 pad 2: /D2+ -> VCC
- D3 pad 1: /KANA_LED_BUFFERED -> Net-(D3-Pad1)
- D3 pad 2: /D3+ -> VCC
- J1 pad 1: /COLUMN0_BUF -> /COL0_BUF
- J1 pad 5: /COLUMN2_BUF -> /COL2_BUF
- J1 pad 9: /COLUMN4_BUF -> /COL4_BUF
- R1 pad 1: VCC -> GND
- R1 pad 2: /D1+ -> Net-(D1-Pad1)
- R2 pad 1: VCC -> Net-(R2-Pad1)
- R2 pad 2: /D2+ -> Net-(D2-Pad1)
- R3 pad 1: VCC -> Net-(R3-Pad1)
- R3 pad 2: /D3+ -> Net-(D3-Pad1)
- RN1 pad 3: /COLUMN0 -> /COL0
- RN1 pad 4: /COLUMN2 -> /COL2
- RN1 pad 5: /COLUMN4 -> /COL4
- SW1 pad 2: /COLUMN0 -> /COL0
- SW10 pad 2: /COLUMN0 -> /COL0
- SW2 pad 2: /COLUMN0 -> /COL0
- SW20 pad 2: /COLUMN2 -> /COL2
- SW21 pad 2: /COLUMN2 -> /COL2
- SW22 pad 2: /COLUMN2 -> /COL2
- SW23 pad 2: /COLUMN2 -> /COL2
- SW24 pad 2: /COLUMN2 -> /COL2
- SW25 pad 2: /COLUMN2 -> /COL2
- SW26 pad 2: /COLUMN2 -> /COL2
- SW27 pad 2: /COLUMN2 -> /COL2
- SW28 pad 2: /COLUMN2 -> /COL2
- SW3 pad 2: /COLUMN0 -> /COL0
- SW38 pad 2: /COLUMN4 -> /COL4
- SW39 pad 2: /COLUMN4 -> /COL4
- SW4 pad 2: /COLUMN0 -> /COL0
- SW40 pad 2: /COLUMN4 -> /COL4
- SW41 pad 2: /COLUMN4 -> /COL4
- SW42 pad 2: /COLUMN4 -> /COL4
- SW43 pad 2: /COLUMN4 -> /COL4
- SW44 pad 2: /COLUMN4 -> /COL4
- SW45 pad 2: /COLUMN4 -> /COL4
- SW46 pad 2: /COLUMN4 -> /COL4
- SW5 pad 2: /COLUMN0 -> /COL0
- SW6 pad 2: /COLUMN0 -> /COL0
- SW7 pad 2: /COLUMN0 -> /COL0
- SW8 pad 2: /COLUMN0 -> /COL0
- SW9 pad 2: /COLUMN0 -> /COL0
- U1 pad 1: /ROW0 -> /COL4
- U1 pad 10: /ROW8 -> Net-(R2-Pad1)
- U1 pad 11: Net-(U1-Pad11) -> /KANA_LED
- U1 pad 12: /ROW_D -> Net-(R3-Pad1)
- U1 pad 13: /ROW_C -> /CAPS_LED
- U1 pad 14: /ROW_B -> VCC
- U1 pad 2: /ROW1 -> /COL4_BUF
- U1 pad 3: /ROW2 -> /COL2
- U1 pad 4: /ROW3 -> /COL2_BUF
- U1 pad 5: /ROW4 -> /COL0
- U1 pad 6: /ROW5 -> /COL0_BUF
- U1 pad 7: /ROW6_UNBUF -> GND
- U1 pad 8: GND -> /ROW6
- U1 pad 9: /ROW7 -> /ROW6_UNBUF
- U2 pad 1: /COLUMN4 -> /ROW0
- U2 pad 10: /KANA_LED_BUFFERED -> /ROW8
- U2 pad 11: /KANA_LED -> unconnected-(U2-Pad11)
- U2 pad 12: /CAPS_LED_BUFFERED -> /ROW_D
- U2 pad 13: /CAPS_LED -> /ROW_C
- U2 pad 14: VCC -> /ROW_B
- U2 pad 2: /COLUMN4_BUF -> /ROW1
- U2 pad 3: /COLUMN2 -> /ROW2
- U2 pad 4: /COLUMN2_BUF -> /ROW3
- U2 pad 5: /COLUMN0 -> /ROW4
- U2 pad 6: /COLUMN0_BUF -> /ROW5
- U2 pad 7: GND -> /ROW6_UNBUF
- U2 pad 8: /ROW6 -> GND
- U2 pad 9: /ROW6_UNBUF -> /ROW7
Routing:
- net GND: track 0.00 -> 827.5 mm
- net /COL1: track 0.00 -> 562.5 mm, vias 0 -> 2
- net /COL5: track 0.00 -> 562.0 mm, vias 0 -> 3
- net /COL7: track 0.00 -> 553.2 mm, vias 0 -> 2
- net /COL4: track 0.00 -> 549.0 mm, vias 0 -> 2
- net /COL0: track 0.00 -> 534.0 mm
- net /COL2: track 0.00 -> 527.4 mm, vias 0 -> 3
- net /COL6: track 0.00 -> 526.9 mm, vias 0 -> 2
- net /ROW7: track 0.00 -> 513.0 mm, vias 0 -> 1
- net /COL3: track 0.00 -> 471.4 mm, vias 0 -> 2
- net /ROW8: track 0.00 -> 470.0 mm
- net /ROW2: track 0.00 -> 369.7 mm, vias 0 -> 2
- net /ROW4: track 0.00 -> 285.1 mm, vias 0 -> 1
- net /ROW6: track 0.00 -> 280.6 mm
- net /SHIFT: track 0.00 -> 255.9 mm
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- added copper zone on B.Cu, net GND
- added copper zone on F.Cu, net GND
Other:
- board size 333.4 x 124.5 mm -> 333.4 x 123.8 mm
- board text added: "'"
- board text added: ","
- board text added: "-"
- board text added: "."
- board text added: "/"
- board text added: "0"
- board text added: "1"
- board text added: "2"
- board text added: "3"
- board text added: "330"
- board text added: "4"
- board text added: "5"
- board text added: "6"
- board text added: "7"
- board text added: "74LS07"
- board text added: "74LS145"
- board text added: "8"
- board text added: "9"
- board text added: ";"
- board text added: "="
- board text added: "A"
- board text added: "B"
- board text added: "BACKSPACE"
- board text added: "C"
- board text added: "CAPS"
- board text added: "CTRL"
- board text added: "D"
- board text added: "DEAD"
- board text added: "DELETE"
- board text added: "DOWN"
- board text added: "E"
- board text added: "ESC"
- board text added: "F"
- board text added: "F1"
- board text added: "F2"
- board text added: "F3"
- board text added: "F4"
- board text added: "F5"
- board text added: "Frédéric Segard"
- board text added: "G"
- board text added: "GRAPH"
- board text added: "H"
- board text added: "HOME"
- board text added: "I"
- board text added: "INSERT"
- board text added: "J"
- board text added: "K"
- board text added: "KANA"
- board text added: "L"
- board text added: "LEFT"
- board text added: "M"
- board text added: "N"
- board text added: "O"
- board text added: "P"
- board text added: "Q"
- board text added: "R"
- board text added: "RETURN"
- board text added: "RIGHT"
- board text added: "Rev 1.0"
- board text added: "S"
- board text added: "SELECT"
- board text added: "SHIFT"
- board text added: "SPACE"
- board text added: "STOP"
- board text added: "T"
- board text added: "TAB"
- board text added: "U"
- board text added: "UP"
- board text added: "V"
- board text added: "W"
- board text added: "X"
- board text added: "Y"
- board text added: "Z"
- board text added: "ZedEighty Project - MSX compatible keyboard - based off Sergey Kiselev's design"
- board text added: "["
- board text added: "\"
- board text added: "]"
- board text added: "youtube.com/@microhobbyist"
- board text added: "~"
- board text removed: "github.com/skiselev/omega www.malinov.com"
