File: Part 7 - Keyboard/Part 7 - Keyboard.kicad_sch (KiCad schematic)
At the start: 96 parts, among them J1 KEYBOARD, SW1 SHIFT, SW10 SPACE, SW11 1, SW12 9, SW13 TILDE, SW14 D, SW15 L, SW16 T, SW17 CTRL, SW18 F5/F10, SW19 HOME/CLS, SW2 0, SW20 2, SW21 MINUS, SW22 COMMA, SW23 E, SW24 M, SW25 U, SW26 GRAPH, SW27 ESC, SW28 INSERT, SW29 3, SW3 8, SW30 EQUALS, SW31 PERIOD, SW32 F, SW33 N, SW34 V, SW35 CAPS_LOCK, SW36 TAB, SW37 DELETE, SW38 4, SW39 BACK_SLASH, SW4 QUOTE, SW40 SLASH, SW41 G, SW42 O, SW43 W, SW44 CODE/KANA, SW45 STOP, SW46 LEFT, SW47 5, SW48 LEFT_BRACKET, SW49 DEAD, SW5 C, SW50 H, SW51 P, SW52 X, SW53 F1/F6, SW54 BACK_SPACE, SW55 UP, SW56 6, SW57 RIGHT_BRACKET, SW58 A, SW59 I, SW6 K, SW60 Q, SW61 Y, SW62 F2/F7, SW63 SELECT, SW64 DOWN, SW65 7, SW66 SEMICOLON, SW67 B, SW68 J, SW69 R, SW7 S, SW70 Z, SW71 F3/F8, SW72 RETURN, SW73 RIGHT, SW8 SHIFT, SW9 F4/F9, U1 74LS07, U2 74LS145

Commit message: Added Keyboard, and minor fixes
Parts:
- H1: value MountingHole_Pad -> MH; footprint MountingHole:MountingHole_3.2mm_M3 -> MountingHole:MountingHole_3.2mm_M3_Pad_Via
- H2, H3, H4, H5, H6, H7: footprint MountingHole:MountingHole_3.2mm_M3 -> MountingHole:MountingHole_3.2mm_M3_Pad_Via
- J1: footprint Connector_PinSocket_2.54mm:PinSocket_2x08_P2.54mm_Horizontal -> Connector_PinSocket_2.54mm:PinSocket_2x08_P2.54mm_Vertical
- SW1: footprint 0_Z80_Library:SW_Cherry_MX_PCB_2.75u -> 0_Z80_Library:SW_Cherry_MX_2.75u_PCB
- SW10: footprint 0_Z80_Library:SW_Cherry_MX_PCB_6.25u -> 0_Z80_Library:SW_Cherry_MX_6.25u_PCB
- SW11, SW12, SW13, SW14, SW15, SW16, SW18, SW19, SW2, SW20, SW21, SW22, SW23, SW24, SW25, SW27, SW28, SW29, SW3, SW31, SW32, SW33, SW34, SW37, SW38, SW4, SW40, SW41, SW42, SW43, SW45, SW46, SW47, SW5, SW50, SW51, SW52, SW53, SW55, SW56, SW58, SW59, SW6, SW60, SW61, SW62, SW64, SW65, SW66, SW67, SW68, SW69, SW7, SW70, SW71, SW73, SW9: footprint 0_Z80_Library:SW_Cherry_MX_PCB_1.00u -> 0_Z80_Library:SW_Cherry_MX_1.00u_PCB
- SW17, SW26, SW44, SW49, SW63: footprint 0_Z80_Library:SW_Cherry_MX_PCB_1.25u -> 0_Z80_Library:SW_Cherry_MX_1.25u_PCB
- SW30: value EQUALS -> EQUAL; footprint 0_Z80_Library:SW_Cherry_MX_PCB_1.00u -> 0_Z80_Library:SW_Cherry_MX_1.00u_PCB
- SW35: value CAPS_LOCK -> CAPS LOCK; footprint 0_Z80_Library:SW_Cherry_MX_PCB_1.75u -> 0_Z80_Library:SW_Cherry_MX_1.75u_PCB
- SW36: footprint 0_Z80_Library:SW_Cherry_MX_PCB_1.50u -> 0_Z80_Library:SW_Cherry_MX_1.50u_PCB
- SW39: value BACK_SLASH -> BACKSLASH; footprint 0_Z80_Library:SW_Cherry_MX_PCB_1.50u -> 0_Z80_Library:SW_Cherry_MX_1.50u_PCB
- SW48: value LEFT_BRACKET -> LEFT BRACKET; footprint 0_Z80_Library:SW_Cherry_MX_PCB_1.00u -> 0_Z80_Library:SW_Cherry_MX_1.00u_PCB
- SW54: value BACK_SPACE -> BACKSPACE; footprint 0_Z80_Library:SW_Cherry_MX_PCB_2.00u -> 0_Z80_Library:SW_Cherry_MX_2.00u_PCB
- SW57: value RIGHT_BRACKET -> RIGHT BRACKET; footprint 0_Z80_Library:SW_Cherry_MX_PCB_1.00u -> 0_Z80_Library:SW_Cherry_MX_1.00u_PCB
- SW72, SW8: footprint 0_Z80_Library:SW_Cherry_MX_PCB_2.25u -> 0_Z80_Library:SW_Cherry_MX_2.25u_PCB
Connections:
- net GND: now also R1.1; no longer D1.1 (K)
- net VCC: now also D1.2 (A), D2.2 (A), D3.2 (A); no longer R1.2, R2.2, R3.2
- net at U1.10: now also R2.1; no longer D2.1 (K)
- net at R3.1: now also U1.12; no longer D3.2 (A)
- net at D3.1 (K): now also R3.2; no longer U1.12
- new net: D1.1 (K), R1.2
- new net: D2.1 (K), R2.2
Other:
- moved on the sheet: D1, D2, D3, R1, R2, R3
